File: quadstep-v11assembly.sch (EAGLE design)
At the start: 120 parts, among them IC2 PIC18F2455_28W, U1 A4983, U2 A4983, U3 A4983, U4 A4983, X1 MSTBA4, X2 MSTBA4, X3 MSTBA4, X4 MSTBA4, X6 ICSP-5

Commit message: Layout ....
Parts:
- removed JP22: (no value), SparkFun:M08
- added JP1: (no value), pinhead:PINHD-1X10
- added JP2, JP3: (no value), pinhead:PINHD-2X6
- added X10, X7, X8, X9: 22-23-2041, con-molex:22-23-2041
- added X11: MSTBA4, con-phoenix-508:MSTBA4
Connections:
- removed net DOUT1: IC2.RC6/TX/CK
- removed net DOUT2: IC2.RB4/AN11/KBI0/CSSPP
- removed net IN3: IC2.RA2/AN2/VREF-/CVREF
- removed net IN4: IC2.RA3/AN3/VREF+
- removed net RL1: IC2.RA5/AN4/!SS!/HLVDIN/C2OUT
- removed net RL2: IC2.RA4/T0CKI/CIOUT/RCV
- removed net RL3: IC2.RC2/CCP1/P1A
- removed net RL4: IC2.RC1/T1OSI/ICCP2/!UOE
- removed net SCLK1: IC2.RC7/RX/DT/SDO
- removed net SCLK2: IC2.RB5/KBI1/PGM
- new net N$55: JP1.1
- new net N$56: JP1.2
- new net N$57: JP1.3
- new net N$58: JP1.4
- new net N$59: JP1.5
- new net N$60: JP1.6
- new net N$61: JP1.7
- new net N$62: JP1.8
- new net N$63: JP1.9
- new net N$64: JP1.10
- net DIR-1: no longer IC2.RA0/AN0
- net LED: no longer IC2.RB0/AN12/INT0/LFT0/SDI/SDA
- net STP-1: no longer IC2.RA1/AN1
Changed lines of the file:
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@@
 <part name="TP4" library="SparkFun" deviceset="TEST-POINT" device="3X5"/>
 <part name="JP21" library="SparkFun" deviceset="M02" device="PTH"/>
-<part name="JP22" library="SparkFun" deviceset="M08" device=""/>
 <part name="GND33" library="SparkFun" deviceset="GND" device=""/>
 <part name="GND34" library="SparkFun" deviceset="GND" device=""/>
@@
 <part name="R32" library="SparkFun" deviceset="RESISTOR" device="0603-RES" value="10k"/>
 <part name="FRAME5" library="frames" deviceset="DINA4_L" device=""/>
+<part name="X7" library="con-molex" deviceset="22-23-2041" device=""/>
+<part name="X8" library="con-molex" deviceset="22-23-2041" device=""/>
+<part name="X9" library="con-molex" deviceset="22-23-2041" device=""/>
+<part name="X10" library="con-molex" deviceset="22-23-2041" device=""/>
+<part name="X11" library="con-phoenix-508" deviceset="MSTBA4" device=""/>
+<part name="JP1" library="pinhead" deviceset="PINHD-1X10" device=""/>
+<part name="JP2" library="pinhead" deviceset="PINHD-2X6" device=""/>
+<part name="JP3" library="pinhead" deviceset="PINHD-2X6" device=""/>
 </parts>
 <sheets>
@@
 <instance part="P+36" gate="G$1" x="223.52" y="124.46"/>
 <instance part="JP21" gate="G$1" x="33.02" y="27.94" rot="MR180"/>
-<instance part="JP22" gate="G$1" x="246.38" y="116.84"/>
 <instance part="GND61" gate="1" x="101.6" y="17.78" rot="MR0"/>
 <instance part="C30" gate="G$1" x="101.6" y="25.4" smashed="yes" rot="MR180">
@@
 </instance>
 <instance part="IC2" gate="G$1" x="96.52" y="147.32"/>
+<instance part="X7" gate="-1" x="17.78" y="111.76"/>
+<instance part="X7" gate="-2" x="17.78" y="109.22"/>
+<instance part="X7" gate="-3" x="17.78" y="106.68"/>
+<instance part="X7" gate="-4" x="17.78" y="104.14"/>
+<instance part="X8" gate="-1" x="35.56" y="111.76"/>
+<instance part="X8" gate="-2" x="35.56" y="109.22"/>
+<instance part="X8" gate="-3" x="35.56" y="106.68"/>
+<instance part="X8" gate="-4" x="35.56" y="104.14"/>
+<instance part="X9" gate="-1" x="50.8" y="111.76"/>
+<instance part="X9" gate="-2" x="50.8" y="109.22"/>
+<instance part="X9" gate="-3" x="50.8" y="106.68"/>
+<instance part="X9" gate="-4" x="50.8" y="104.14"/>
+<instance part="X10" gate="-1" x="66.04" y="111.76"/>
+<instance part="X10" gate="-2" x="66.04" y="109.22"/>
+<instance part="X10" gate="-3" x="66.04" y="106.68"/>
+<instance part="X10" gate="-4" x="66.04" y="104.14"/>
+<instance part="X11" gate="-1" x="22.86" y="58.42"/>
+<instance part="X11" gate="-2" x="22.86" y="53.34"/>
+<instance part="X11" gate="-3" x="22.86" y="48.26"/>
+<instance part="X11" gate="-4" x="22.86" y="43.18"/>
+<instance part="JP1" gate="A" x="248.92" y="114.3"/>
+<instance part="JP2" gate="A" x="236.22" y="147.32"/>
+<instance part="JP3" gate="A" x="160.02" y="167.64"/>
 </instances>
 <busses>
@@
 </segment>
 </net>
-<net name="DOUT2" class="0">
-<segment>
-<wire x1="134.62" y1="154.94" x2="137.16" y2="154.94" width="0.1524" layer="91"/>
-<label x="137.16" y="154.94" size="1.27" layer="95" xref="yes"/>
-<pinref part="IC2" gate="G$1" pin="RB4/AN11/KBI0/CSSPP"/>
-<junction x="134.62" y="154.94"/>
-</segment>
-</net>
-<net name="SCLK1" class="0">
-<segment>
-<wire x1="134.62" y1="137.16" x2="137.16" y2="137.16" width="0.1524" layer="91"/>
-<label x="137.16" y="137.16" size="1.016" layer="95" rot="MR180" xref="yes"/>
-<pinref part="IC2" gate="G$1" pin="RC7/RX/DT/SDO"/>
-<junction x="134.62" y="137.16"/>
-</segment>
-</net>
-<net name="DOUT1" class="0">
-<segment>
-<wire x1="134.62" y1="134.62" x2="137.16" y2="134.62" width="0.1524" layer="91"/>
-<label x="137.16" y="134.62" size="1.016" layer="95" rot="MR180" xref="yes"/>
-<pinref part="IC2" gate="G$1" pin="RC6/TX/CK"/>
-<junction x="134.62" y="134.62"/>
-</segment>
-</net>
 <net name="N$54" class="0">
 <segment>
@@
 <wire x1="124.46" y1="63.5" x2="121.92" y2="63.5" width="0.1524" layer="91"/>
 <label x="121.92" y="63.5" size="1.016" layer="95" rot="R180" xref="yes"/>
-</segment>
-<segment>
-<wire x1="137.16" y1="144.78" x2="134.62" y2="144.78" width="0.1524" layer="91"/>
-<label x="137.16" y="144.78" size="1.27" layer="95" xref="yes"/>
-<pinref part="IC2" gate="G$1" pin="RB0/AN12/INT0/LFT0/SDI/SDA"/>
-<junction x="134.62" y="144.78"/>
-</segment>
-</net>
-<net name="SCLK2" class="0">
-<segment>
-<wire x1="134.62" y1="157.48" x2="137.16" y2="157.48" width="0.1524" layer="91"/>
-<label x="137.16" y="157.48" size="1.27" layer="95" xref="yes"/>
-<pinref part="IC2" gate="G$1" pin="RB5/KBI1/PGM"/>
-<junction x="134.62" y="157.48"/>
-</segment>
-</net>
-<net name="RL1" class="0">
-<segment>
-<wire x1="58.42" y1="147.32" x2="55.88" y2="147.32" width="0.1524" layer="91"/>
-<label x="55.88" y="147.32" size="1.27" layer="95" rot="R180" xref="yes"/>
-<pinref part="IC2" gate="G$1" pin="RA5/AN4/!SS!/HLVDIN/C2OUT"/>
-</segment>
-</net>
-<net name="RL2" class="0">
-<segment>
-<wire x1="55.88" y1="149.86" x2="58.42" y2="149.86" width="0.1524" layer="91"/>
-<label x="55.88" y="149.86" size="1.27" layer="95" rot="R180" xref="yes"/>
-<pinref part="IC2" gate="G$1" pin="RA4/T0CKI/CIOUT/RCV"/>
-</segment>
-</net>
-<net name="RL3" class="0">
-<segment>
-<wire x1="55.88" y1="132.08" x2="58.42" y2="132.08" width="0.1524" layer="91"/>
-<label x="55.88" y="132.08" size="1.27" layer="95" rot="R180" xref="yes"/>
-<pinref part="IC2" gate="G$1" pin="RC2/CCP1/P1A"/>
-</segment>
-</net>
-<net name="RL4" class="0">
-<segment>
-<wire x1="55.88" y1="134.62" x2="58.42" y2="134.62" width="0.1524" layer="91"/>
-<label x="55.88" y="134.62" size="1.27" layer="95" rot="R180" xref="yes"/>
-<pinref part="IC2" gate="G$1" pin="RC1/T1OSI/ICCP2/!UOE"/>
-</segment>
-</net>
-<net name="DIR-1" class="0">
-<segment>
-<wire x1="58.42" y1="160.02" x2="55.88" y2="160.02" width="0.1524" layer="91"/>
-<label x="55.88" y="160.02" size="1.27" layer="95" rot="MR0" xref="yes"/>
-<pinref part="IC2" gate="G$1" pin="RA0/AN0"/>
-</segment>
-</net>
-<net name="STP-1" class="0">
-<segment>
-<wire x1="58.42" y1="157.48" x2="55.88" y2="157.48" width="0.1524" layer="91"/>
-<label x="55.88" y="157.48" size="1.27" layer="95" rot="MR0" xref="yes"/>
-<pinref part="IC2" gate="G$1" pin="RA1/AN1"/>
-</segment>
-</net>
-<net name="IN3" class="0">
-<segment>
-<wire x1="58.42" y1="154.94" x2="55.88" y2="154.94" width="0.1524" layer="91"/>
-<label x="55.88" y="154.94" size="1.27" layer="95" rot="MR0" xref="yes"/>
-<pinref part="IC2" gate="G$1" pin="RA2/AN2/VREF-/CVREF"/>
-</segment>
-</net>
-<net name="IN4" class="0">
-<segment>
-<wire x1="58.42" y1="152.4" x2="55.88" y2="152.4" width="0.1524" layer="91"/>
-<label x="55.88" y="152.4" size="1.27" layer="95" rot="MR0" xref="yes"/>
-<pinref part="IC2" gate="G$1" pin="RA3/AN3/VREF+"/>
 </segment>
 </net>
@@
 </segment>
 </net>
+<net name="N$55" class="0">
+<segment>
+<pinref part="JP1" gate="A" pin="1"/>
+<wire x1="246.38" y1="124.46" x2="241.3" y2="124.46" width="0.1524" layer="91"/>
+</segment>
+</net>
+<net name="N$56" class="0">
+<segment>
+<pinref part="JP1" gate="A" pin="2"/>
+<wire x1="246.38" y1="121.92" x2="241.3" y2="121.92" width="0.1524" layer="91"/>
+</segment>
+</net>
+<net name="N$57" class="0">
+<segment>
+<pinref part="JP1" gate="A" pin="3"/>
+<wire x1="246.38" y1="119.38" x2="241.3" y2="119.38" width="0.1524" layer="91"/>
+</segment>
+</net>
+<net name="N$58" class="0">
+<segment>
+<pinref part="JP1" gate="A" pin="4"/>
+<wire x1="246.38" y1="116.84" x2="241.3" y2="116.84" width="0.1524" layer="91"/>
+</segment>
+</net>
+<net name="N$59" class="0">
+<segment>
+<pinref part="JP1" gate="A" pin="5"/>
+<wire x1="246.38" y1="114.3" x2="241.3" y2="114.3" width="0.1524" layer="91"/>
+</segment>
+</net>
+<net name="N$60" class="0">
+<segment>
+<pinref part="JP1" gate="A" pin="6"/>
+<wire x1="246.38" y1="111.76" x2="241.3" y2="111.76" width="0.1524" layer="91"/>
+</segment>
+</net>
+<net name="N$61" class="0">
+<segment>
+<pinref part="JP1" gate="A" pin="7"/>
+<wire x1="246.38" y1="109.22" x2="241.3" y2="109.22" width="0.1524" layer="91"/>
+</segment>
+</net>
+<net name="N$62" class="0">
+<segment>
+<pinref part="JP1" gate="A" pin="8"/>
+<wire x1="246.38" y1="106.68" x2="241.3" y2="106.68" width="0.1524" layer="91"/>
+</segment>
+</net>
+<net name="N$63" class="0">
+<segment>
+<pinref part="JP1" gate="A" pin="9"/>
+<wire x1="246.38" y1="104.14" x2="241.3" y2="104.14" width="0.1524" layer="91"/>
+</segment>
+</net>
+<net name="N$64" class="0">
+<segment>
+<pinref part="JP1" gate="A" pin="10"/>
+<wire x1="246.38" y1="101.6" x2="241.3" y2="101.6" width="0.1524" layer="91"/>
+</segment>
+</net>

Commit message: Layout with new TQFP IC
Parts:
- removed C25, C26: 8pF, SparkFun:CAP0603-CAP
- removed C27, C28, C29, C32: 100nF, SparkFun:CAP0805
- removed C30: 10uF, SparkFun:CAP0805
- removed C31: 470uF, SparkFun:CAP_POLG
- removed C41: 0.1uF, SparkFun:CAP0402-CAP
- removed C44: 1uF, SparkFun:CAP0805
- removed IC1: (no value), SparkFun:V_REG_LM1117SOT223
- removed IC2: PIC18F2455_28W, microchip:PIC18F2455_28W
- removed JP21: (no value), SparkFun:M02PTH
- removed JP3: (no value), pinhead:PINHD-2X6
- removed LED5: red, SparkFun:LED0603
- removed R36: 330, SparkFun:RESISTOR0402-RES
- removed R37: 10k, SparkFun:RESISTOR
- removed U$6: CRYSTAL-SMD- 12MHz, crystal:CRYSTAL-SMD
- removed X10, X7, X8, X9: 22-23-2041, con-molex:22-23-2041
- removed X5: (no value), con-berg:PN61729
- removed X6: ICSP-5, ICSP:ICSP-5
- added C33: 10uF, SparkFun:CAP0805
- added C34, C36, C37, C38, C39: 100nF, SparkFun:CAP0805
- added C35: 470uF, SparkFun:CAP_POLG
- added C40, C42: 8pF, SparkFun:CAP0603-CAP
- added IC3: NCP1117ST50T3G, SparkFun:V_REG_LM1117SOT223
- added IC6: PIC18F4550_TQFP, microchip:PIC18F4550_TQFP
- added JP4, JP5: (no value), pinhead:PINHD-2X5
- added LED2, LED3: (no value), led:LEDCHIPLED_0805
- added R49, R50, R51: 10k, SparkFun:RESISTOR
- added U$4: CRYSTAL-SMD- 12MHz, crystal:CRYSTAL-SMD
- added X12: USB B, con-berg:PN61729
- added X14: ICSP-5, ICSP:ICSP-5
- JP2: device pinhead:PINHD-2X6 -> pinhead:PINHD-2X3
Connections:
- removed net LED: R33.2
- removed net VDD: IC2.VDD, R34.1, X6.VDD
- new net LED1: IC6.RB4/AN11/KBI0/CSSPP, R33.2
- new net LED2: IC6.RB5/KBI1/PGM, R34.2
- new net N$65: IC6.RA0/AN0, JP5.8
- new net N$66: IC6.RA1/AN1, JP5.7
- new net N$67: IC6.RA2/AN2/VREF-/CVREF, JP5.6
- new net N$68: IC6.RA3/AN3/VREF+, JP5.5
- new net N$69: IC6.RA4/T0CKI/CIOUT/RCV, JP5.3
- new net N$70: IC6.RA5/AN4/!SS!/HLVDIN/C2OUT, JP5.4
- new net N$71: IC6.RE0/AN5/CK1SPP, JP5.1
- new net N$72: IC6.RE1/AN6/CK2SPP, JP5.2
- new net N$73: LED2.A, R34.1
- new net N$74: IC6.RC1/T1OSI/ICCP2/!UOE, JP2.2
- new net N$75: IC6.RC2/CCP1/P1A, JP2.4
- new net N$76: IC6.RC0/TIOSO/T13CKI, JP2.3
- new net N$77: IC6.RE2/AN7/OESPP, JP2.1
- net !MCLR: now also IC6.!MCLR!/VPP/RE3, R51.2, X14.VPP; no longer IC2.!MCLR!/VPP/RE3, R34.2, X6.VPP
- net D+: now also IC6.RC5/D+/VP, X12.3; no longer IC2.RC5/D+/VP, X5.3
- net D-: now also IC6.RC4/D-/VM, X12.2; no longer IC2.RC4/D-/VM, X5.2
- net DIR-1: now also IC6.RD0/SPP0, JP4.7
- net DIR-2: now also IC6.RD1/SPP1, JP4.5
- net DIR-3: now also IC6.RD2/SPP2, JP4.3
- net DIR-4: now also IC6.RD3/SPP3, JP4.1
- net EN: now also IC6.RC7/RX/DT/SDO
- net GND: now also C33.1, C34.1, C35.-, C36.1, C37.2, C38.2, C39.2, C40.2, C42.2, IC3.ADJ, IC6.VSS, IC6.VSS@1, JP2.5, JP4.10, JP5.9, LED2.C, LED3.C, R50.2, U$4.GND, U$4.GND2, X12.4, X14.VSS; no longer C25.2, C26.2, C27.1, C28.1, C29.1, C30.1, C31.-, C32.1, C41.2, C44.2, IC1.ADJ, IC2.VSS, IC2.VSS@1, JP21.2, R36.1, R37.2, U$6.GND, U$6.GND2, X5.4, X6.VSS
- net N$27: now also LED3.A, R35.1; no longer LED5.C, R36.2
- net OSC1: now also C42.1, IC6.OSC1/CLKI, U$4.OSC2; no longer C26.1, IC2.OSC1/CLKI, U$6.OSC2
- net OSC2: now also C40.1, IC6.RA6/OSC2/CLKO, U$4.OSC1; no longer C25.1, IC2.RA6/OSC2/CLKO, U$6.OSC1
- net PGC: now also IC6.RB6/KBI2/PGC, X14.PGC; no longer IC2.RB6/KBI2/PGC, X6.PGC
- net PGD: now also IC6.RB7/BKI3/PGD, X14.PGD; no longer IC2.RB7/BKI3/PGD, X6.PGD
- net SLP: now also IC6.RD4/SPP4
- net STP-1: now also IC6.RB0/AN12/INT0/LFT0/SDI/SDA, JP4.8
- net STP-2: now also IC6.RB1/AN10/INT1/SCK/SCL, JP4.6
- net STP-3: now also IC6.RB2/AN8/INT2/VMO, JP4.4
- net STP-4: now also IC6.RB3/AN9/CCP2/VPO, JP4.2
- net USB_SENSE: now also IC6.RC6/TX/CK, R49.2; no longer IC2.RB1/AN10/INT1/SCK/SCL, R35.2
- net VBUS: now also R49.1, R50.1, X12.1; no longer R35.1, R37.1, X5.1
- net VCC: now also C35.+, C36.2, IC3.IN, X11-1.1, X11-2.1; no longer C31.+, C32.2, IC1.IN, JP21.1
- net VOUT: now also C33.2, C34.2, IC3.OUT, IC3.OUT@1, IC6.VDD, IC6.VDD@1, JP2.6, JP4.9, JP5.10, R35.2, R51.1, X14.VDD; no longer C30.2, C41.1, C44.1, IC1.OUT, IC1.OUT@1, LED5.A
- net VUSB: now also C37.1, C38.1, C39.1, IC6.VUSB; no longer C27.2, C28.2, C29.2, IC2.VUSB
Other:
- note added: "by Arthur Benemann"
