File: QuadStepDriver.sch (EAGLE design)
At the start: 124 parts, among them IC3 NCP1117ST50T3G, IC6 PIC18F4550_TQFP, U1 A4983, U2 A4983, U3 A4983, U4 A4983, X1 MSTBA4, X11 MSTBA4, X12 USB B, X14 ICSP-5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

Commit message: Just cleaning up the schematic
Parts:
- removed JP1: (no value), pinhead:PINHD-1X10
- removed JP11: STAND-OFF, SparkFun:STAND-OFF
Connections:
- net N$65 renamed RA0
- net N$66 renamed RA1
- net N$67 renamed RA2
- net N$68 renamed RA3
- net N$69 renamed RA4
- net N$70 renamed RA5
- net N$71 renamed RE0
- net N$72 renamed RE1
- net N$74 renamed RC1
- net N$75 renamed RC2
- net N$76 renamed RC0
- net N$77 renamed RE2
- removed net N$56: JP1.2
- removed net N$57: JP1.3
- removed net N$58: JP1.4
- removed net N$59: JP1.5
- removed net N$60: JP1.6
- removed net N$61: JP1.7
- removed net N$62: JP1.8
- removed net N$63: JP1.9
- removed net N$64: JP1.10
- net LED1: no longer R33.2
- net N$55: now also R33.2; no longer JP1.1
- net PGC: no longer IC6.RB6/KBI2/PGC
Other:
- moved on the sheet: C35, C37, C38, C39, C40, C42, IC3, IC6, JP2, JP4, JP5, LED1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

Commit message: PCB: Finalizando Gerbers
Connections:
- removed net N$55: R33.2
- net LED1: now also IC6.RB5/KBI1/PGM, R34.2; no longer IC6.RB4/AN11/KBI0/CSSPP
- net LED2: now also IC6.RB4/AN11/KBI0/CSSPP, R33.2; no longer IC6.RB5/KBI1/PGM, R34.2
Changed lines of the file:
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@@
 <?xml version="1.0" encoding="utf-8"?>
 <!DOCTYPE eagle SYSTEM "eagle.dtd">
-<eagle version="6.1">
+<eagle version="6.4">
 <drawing>
 <settings>
@@
 </segment>
 </net>
-<net name="LED1" class="0">
+<net name="LED2" class="0">
 <segment>
 <wire x1="33.02" y1="132.08" x2="30.48" y2="132.08" width="0.1524" layer="91"/>
 <pinref part="IC6" gate="G$1" pin="RB4/AN11/KBI0/CSSPP"/>
 <label x="30.48" y="132.08" size="1.27" layer="95" rot="R180" xref="yes"/>
+</segment>
+<segment>
+<pinref part="R33" gate="G$1" pin="2"/>
+<wire x1="190.5" y1="78.74" x2="187.96" y2="78.74" width="0.1524" layer="91"/>
+<label x="187.96" y="78.74" size="1.016" layer="95" rot="R180" xref="yes"/>
 </segment>
 </net>
@@
 </segment>
 </net>
-<net name="LED2" class="0">
+<net name="LED1" class="0">
 <segment>
 <pinref part="R34" gate="G$1" pin="2"/>
@@
 </segment>
 </net>
-<net name="N$55" class="0">
-<segment>
-<pinref part="R33" gate="G$1" pin="2"/>
-<wire x1="190.5" y1="78.74" x2="187.96" y2="78.74" width="0.1524" layer="91"/>
-<label x="187.96" y="78.74" size="1.016" layer="95" rot="R180" xref="yes"/>
-</segment>
-</net>

Commit message: Changing some components values, and organizing component values placement
Parts:
- R33, R34, R35: value 10k -> 330R
Changed lines of the file:
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@@
 <part name="FRAME1" library="frames" deviceset="DINA4_L" device=""/>
 <part name="FRAME2" library="frames" deviceset="DINA4_L" device=""/>
-<part name="R33" library="SparkFun" deviceset="RESISTOR" device="" value="10k"/>
+<part name="R33" library="SparkFun" deviceset="RESISTOR" device="" value="330R"/>
 <part name="LED1" library="led" deviceset="LED" device="CHIPLED_0805"/>
 <part name="GND49" library="supply1" deviceset="GND" device=""/>
@@
 <part name="JP4" library="pinhead" deviceset="PINHD-2X5" device=""/>
 <part name="JP5" library="pinhead" deviceset="PINHD-2X5" device=""/>
-<part name="R34" library="SparkFun" deviceset="RESISTOR" device="" value="10k"/>
+<part name="R34" library="SparkFun" deviceset="RESISTOR" device="" value="330R"/>
 <part name="LED2" library="led" deviceset="LED" device="CHIPLED_0805"/>
 <part name="GND3" library="supply1" deviceset="GND" device=""/>
-<part name="R35" library="SparkFun" deviceset="RESISTOR" device="" value="10k"/>
+<part name="R35" library="SparkFun" deviceset="RESISTOR" device="" value="330R"/>
 <part name="LED3" library="led" deviceset="LED" device="CHIPLED_0805"/>
 <part name="GND10" library="supply1" deviceset="GND" device=""/>

Commit message: Fixing some unconneted routes from board REV1.
PGC and power input GND are now connected.
Connections:
- net GND: now also X11-3.1, X11-4.1
- net PGC: now also IC6.RB6/KBI2/PGC
Changed lines of the file:
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@@
 <part name="GND10" library="supply1" deviceset="GND" device=""/>
 <part name="JP2" library="pinhead" deviceset="PINHD-2X3" device=""/>
+<part name="GND32" library="supply1" deviceset="GND" device=""/>
 </parts>
 <sheets>
@@
 <instance part="GND10" gate="1" x="210.82" y="86.36" rot="MR270"/>
 <instance part="JP2" gate="A" x="195.58" y="111.76"/>
+<instance part="GND32" gate="1" x="35.56" y="12.7" rot="MR0"/>
 </instances>
 <busses>
@@
 <pinref part="GND10" gate="1" pin="GND"/>
 <pinref part="LED3" gate="G$1" pin="C"/>
+</segment>
+<segment>
+<pinref part="X11" gate="-3" pin="1"/>
+<wire x1="33.02" y1="20.32" x2="35.56" y2="20.32" width="0.1524" layer="91"/>
+<wire x1="35.56" y1="20.32" x2="35.56" y2="15.24" width="0.1524" layer="91"/>
+<pinref part="X11" gate="-4" pin="1"/>
+<wire x1="35.56" y1="15.24" x2="33.02" y2="15.24" width="0.1524" layer="91"/>
+<pinref part="GND32" gate="1" pin="GND"/>
+<junction x="35.56" y="15.24"/>
 </segment>
 </net>
@@
 <net name="PGC" class="0">
 <segment>
+<wire x1="30.48" y1="127" x2="33.02" y2="127" width="0.1524" layer="91"/>
+<pinref part="IC6" gate="G$1" pin="RB6/KBI2/PGC"/>
+<label x="30.48" y="127" size="1.27" layer="95" rot="R180" xref="yes"/>
+</segment>
+<segment>
 <pinref part="X14" gate="G$1" pin="PGC"/>
